File: RedPink_STM32C09_Board.kicad_pcb (KiCad board)
At the start: 2 copper layers, 80 x 25 mm, 39 parts, among them IC1 STM32C092CBT6, IC3 ATA6561-GAQW-N, IC4 LDLN025M18R, IC5 FT231XS-U, J1 USB4216-03-A, J2 SWD DEBUG, J3 CANBUS, Y1 NX3225GD-8MHZ-STD-CRA-3

Commit message: Updated PCB layout, output connector replaced
1) Removed 5V pin from output pin header
2) Added round corners
3) Replace pin header output
Parts:
- removed J3: CANBUS, Connector_PinHeader_2.54mm:PinHeader_1x04_P2.54mm_Vertical
- added J4: CANBUS, Connector_PinHeader_2.54mm:PinHeader_1x03_P2.54mm_Vertical, F.Cu at (189.5, 70.2)
Routing:
- net 5V: track 103.2 -> 53.4 mm
- net 3V3: track 59.9 -> 64.3 mm
- net VSS: vias 228 -> 272
Other:
- outline, holes or cut-outs redrawn
- board text added: "CANBus USB Adapter Rev 1 Alan R. Montt"
- board text removed: "5V"
- board text removed: "CANBus - USB Adapter Rev 0 Alan R. Montt"
